File: placa_dos_motores.kicad_pcb (KiCad board)
At the start: 2 copper layers, 21 parts, among them J1 Barrel_Jack, J2 Conn_01x04_Female, J3 Conn_01x04_Female, J4 Conn_01x04_Female, J5 Conn_01x04_Female, J6 Conn_01x04_Female, U1 L7805, U2 POLOLU_A4988, U3 POLOLU_A4988, U4 POLOLU_A4988, U5 POLOLU_A4988, U6 Arduino_Nano_R3

Commit message: estado atual e final
Parts:
- added J7: Conn_01x02_Female, Connectors_Terminal_Blocks:TerminalBlock_bornier-2_P5.08mm, F.Cu at (112.5, 50.0)
- moved J6 3.00 mm to (136.0, 50.0)
Connections:
- J6 pad 1: Net-(J6-Pad1) -> VMM
- U3 pad 10: VDD -> Net-(U3-Pad10)
- U3 pad 11: GND -> VDD
- U4 pad 16: GND -> Net-(U4-Pad16)
- U6 pad 21: Net-(U4-Pad15) -> Net-(U4-Pad16)
- U6 pad 22: Net-(U3-Pad16) -> Net-(U4-Pad15)
- U6 pad 23: Net-(U3-Pad15) -> Net-(U3-Pad16)
- U6 pad 24: Net-(J6-Pad1) -> Net-(U3-Pad15)
Routing:
- net Net-(J6-Pad1): track 79.9 -> 0.00 mm
- net Net-(U4-Pad16): track 0.00 -> 40.3 mm
- net GND: track 420.7 -> 447.5 mm
- net VDD: track 282.9 -> 302.0 mm
- net VMM: track 280.7 -> 275.8 mm
- net Net-(J6-Pad4): track 63.2 -> 59.3 mm
- net Net-(J6-Pad3): track 68.9 -> 65.6 mm
- net Net-(J6-Pad2): track 74.4 -> 71.6 mm
- net Net-(U4-Pad15): track 39.0 -> 40.5 mm
- net Net-(U3-Pad15): track 34.9 -> 33.9 mm
- net Net-(U3-Pad16): track 34.9 -> 33.9 mm
