File: placa_dos_motores.sch (KiCad schematic (older format))
At the start: 21 parts, among them J1 Barrel_Jack, J2 Conn_01x04_Female, J3 Conn_01x04_Female, J4 Conn_01x04_Female, J5 Conn_01x04_Female, J6 Conn_01x04_Female, U1 L7805, U2 POLOLU_A4988, U3 POLOLU_A4988, U4 POLOLU_A4988, U5 POLOLU_A4988, U6 Arduino_Nano_R3

Commit message: estado atual e final
Parts:
- added J7: Conn_01x02_Female, Connectors_Terminal_Blocks:TerminalBlock_bornier-2_P5.08mm, symbol Conn_01x02_Female
Connections:
- net GND: now also J7.1 (Pin_1); no longer U3.11 (MS2), U4.16 (DIR)
- net VDD: now also U3.11 (MS2), J7.2 (Pin_2); no longer U3.10 (MS1)
- net VMM: now also J6.1 (Pin_1)
- net at U3.15 (STEP): now also U6.24 (D6); no longer U6.23 (D5)
- net at U3.16 (DIR): now also U6.23 (D5); no longer U6.22 (D4)
- net at U4.15 (STEP): now also U6.22 (D4); no longer U6.21 (D3)
- new net: U4.16 (DIR), U6.21 (D3)
Other:
- moved on the sheet: J6
Changed lines of the file:
@@
 L VDD #PWR014
 U 1 1 5BF87E33
-P 6400 3050
-F 0 "#PWR014" H 6400 2900 50  0001 C CNN
-F 1 "VDD" H 6400 3200 50  0000 C CNN
-F 2 "" H 6400 3050 50  0001 C CNN
-F 3 "" H 6400 3050 50  0001 C CNN
-	1    6400 3050
+P 6400 2950
+F 0 "#PWR014" H 6400 2800 50  0001 C CNN
+F 1 "VDD" H 6400 3100 50  0000 C CNN
+F 2 "" H 6400 2950 50  0001 C CNN
+F 3 "" H 6400 2950 50  0001 C CNN
+	1    6400 2950
 	1    0    0    -1
 $EndComp
@@
 $Comp
 L GND #PWR026
-U 1 1 5BF9BB72
-P 6250 3800
-F 0 "#PWR026" H 6250 3550 50  0001 C CNN
-F 1 "GND" H 6250 3650 50  0000 C CNN
-F 2 "" H 6250 3800 50  0001 C CNN
-F 3 "" H 6250 3800 50  0001 C CNN
-	1    6250 3800
-	1    0    0    -1
-$EndComp
-$Comp
-L GND #PWR027
 U 1 1 5BF9BBFE
 P 6250 5150
-F 0 "#PWR027" H 6250 4900 50  0001 C CNN
+F 0 "#PWR026" H 6250 4900 50  0001 C CNN
 F 1 "GND" H 6250 5000 50  0000 C CNN
 F 2 "" H 6250 5150 50  0001 C CNN
@@
 $EndComp
 $Comp
-L GND #PWR028
+L GND #PWR027
 U 1 1 5BF9C3B2
 P 6250 2450
-F 0 "#PWR028" H 6250 2200 50  0001 C CNN
+F 0 "#PWR027" H 6250 2200 50  0001 C CNN
 F 1 "GND" H 6250 2300 50  0000 C CNN
 F 2 "" H 6250 2450 50  0001 C CNN
@@
 $EndComp
 $Comp
-L GND #PWR029
+L GND #PWR028
 U 1 1 5BF9D408
 P 7900 4200
-F 0 "#PWR029" H 7900 3950 50  0001 C CNN
+F 0 "#PWR028" H 7900 3950 50  0001 C CNN
 F 1 "GND" H 7900 4050 50  0000 C CNN
 F 2 "" H 7900 4200 50  0001 C CNN
@@
 $EndComp
 $Comp
-L VDD #PWR030
+L VDD #PWR029
 U 1 1 5BF9D5A5
 P 7800 1650
-F 0 "#PWR030" H 7800 1500 50  0001 C CNN
+F 0 "#PWR029" H 7800 1500 50  0001 C CNN
 F 1 "VDD" H 7800 1800 50  0000 C CNN
 F 2 "" H 7800 1650 50  0001 C CNN
@@
 $EndComp
 $Comp
-L GND #PWR031
+L GND #PWR030
 U 1 1 5BFE8F59
 P 8500 2000
-F 0 "#PWR031" H 8500 1750 50  0001 C CNN
+F 0 "#PWR030" H 8500 1750 50  0001 C CNN
 F 1 "GND" H 8500 1850 50  0000 C CNN
 F 2 "" H 8500 2000 50  0001 C CNN
@@
 $EndComp
 $Comp
-L GND #PWR032
+L GND #PWR031
 U 1 1 5BFE9662
 P 7450 2000
-F 0 "#PWR032" H 7450 1750 50  0001 C CNN
+F 0 "#PWR031" H 7450 1750 50  0001 C CNN
 F 1 "GND" H 7450 1850 50  0000 C CNN
 F 2 "" H 7450 2000 50  0001 C CNN
@@
 $EndComp
 $Comp
-L GND #PWR033
+L GND #PWR032
 U 1 1 5BFE96A9
 P 7150 2000
-F 0 "#PWR033" H 7150 1750 50  0001 C CNN
+F 0 "#PWR032" H 7150 1750 50  0001 C CNN
 F 1 "GND" H 7150 1850 50  0000 C CNN
 F 2 "" H 7150 2000 50  0001 C CNN
@@
 	1    0    0    -1
 $EndComp
+$Comp
+L Conn_01x04_Female J6
+U 1 1 5BFEA786
+P 10150 3100
+F 0 "J6" H 10150 3300 50  0000 C CNN
+F 1 "Conn_01x04_Female" H 10550 2900 50  0000 C CNN
+F 2 "Connectors_Terminal_Blocks:TerminalBlock_bornier-4_P5.08mm" H 10150 3100 50  0001 C CNN
+F 3 "" H 10150 3100 50  0001 C CNN
+	1    10150 3100
+	1    0    0    -1
+$EndComp
+$Comp
+L GND #PWR033
+U 1 1 5C086770
+P 6250 3800
+F 0 "#PWR033" H 6250 3550 50  0001 C CNN
+F 1 "GND" H 6250 3650 50  0000 C CNN
+F 2 "" H 6250 3800 50  0001 C CNN
+F 3 "" H 6250 3800 50  0001 C CNN
+	1    6250 3800
+	1    0    0    -1
+$EndComp
 Wire Wire Line
 	4000 1700 4200 1700
@@
 Connection ~ 4200 3050
 Wire Wire Line
-	6400 3050 6400 3150
-Wire Wire Line
-	6400 3150 6000 3150
+	6400 2950 6400 3050
+Wire Wire Line
+	6400 3050 6000 3050
 Wire Wire Line
 	6000 2750 6000 2850
@@
 	6100 1200 6000 1200
 Wire Wire Line
-	6250 3800 6250 3750
-Wire Wire Line
-	6250 3750 6100 3750
-Wire Wire Line
-	6100 3900 6000 3900
-Wire Wire Line
 	6250 5150 6250 5100
 Wire Wire Line
@@
 Wire Wire Line
 	6100 4300 6000 4300
-Connection ~ 6100 3900
 Wire Wire Line
 	6100 4400 6000 4400
-Connection ~ 6100 4300
 Wire Wire Line
 	6100 1600 6000 1600
@@
 	6250 2400 6100 2400
 Wire Wire Line
-	6100 2400 6100 3050
-Wire Wire Line
-	6100 2950 6000 2950
-Wire Wire Line
-	6100 3050 6000 3050
-Connection ~ 6100 2950
-Wire Wire Line
 	7900 4050 7900 4200
 Connection ~ 7900 4150
@@
 	6800 1450 9600 1450
 Wire Wire Line
-	6000 4000 7150 4000
-Wire Wire Line
-	7150 4000 7150 4500
+	7150 3900 7150 4500
 Wire Wire Line
 	7150 4500 9400 4500
@@
 	6000 5350 9700 5350
 Wire Wire Line
-	9600 1450 9600 2900
+	9600 1450 9600 3000
 Wire Wire Line
 	7150 1700 7150 1650
@@
 	9400 2700 8950 2700
 Wire Wire Line
-	9600 2900 8950 2900
-Wire Wire Line
-	6900 1350 9300 1350
-Wire Wire Line
-	9300 1350 9300 2800
+	6000 1300 6800 1300
+Wire Wire Line
+	6800 1300 6800 1250
+Wire Wire Line
+	6800 1250 9500 1250
+Wire Wire Line
+	8950 3100 9950 3100
+Wire Wire Line
+	8950 3200 9950 3200
+Wire Wire Line
+	8950 3300 9950 3300
+Wire Wire Line
+	8950 3400 9500 3400
+Wire Wire Line
+	9600 3000 8950 3000
+Wire Wire Line
+	9500 3400 9500 1250
+Wire Wire Line
+	8100 4150 7900 4150
+Wire Wire Line
+	8100 4050 8100 4150
+Wire Wire Line
+	6100 3750 6100 4400
+Wire Wire Line
+	6250 3800 6250 3750
+Wire Wire Line
+	6250 3750 6100 3750
+Connection ~ 6100 4300
+Wire Wire Line
+	6000 3900 7150 3900
+Wire Wire Line
+	6000 4000 7250 4000
+Wire Wire Line
+	7250 4000 7250 4600
+Wire Wire Line
+	7250 4600 9300 4600
+Wire Wire Line
+	9300 4600 9300 2800
 Wire Wire Line
 	9300 2800 8950 2800
 Wire Wire Line
-	6000 1300 6800 1300
-Wire Wire Line
-	6800 1300 6800 1250
-Wire Wire Line
-	6800 1250 9500 1250
-$Comp
-L Conn_01x04_Female J6
-U 1 1 5BFEA786
-P 9200 3100
-F 0 "J6" H 9200 3300 50  0000 C CNN
-F 1 "Conn_01x04_Female" H 9600 2900 50  0000 C CNN
-F 2 "Connectors_Terminal_Blocks:TerminalBlock_bornier-4_P5.08mm" H 9200 3100 50  0001 C CNN
-F 3 "" H 9200 3100 50  0001 C CNN
-	1    9200 3100
-	1    0    0    -1
-$EndComp
-Wire Wire Line
-	9000 3100 8950 3100
-Wire Wire Line
-	8950 3200 9000 3200
-Wire Wire Line
-	9000 3300 8950 3300
-Wire Wire Line
-	8950 3400 9500 3400
-Wire Wire Line
-	8950 3000 9000 3000
-Wire Wire Line
-	9500 3400 9500 1250
-Wire Wire Line
-	8100 4150 7900 4150
-Wire Wire Line
-	8100 4050 8100 4150
-Wire Wire Line
-	6100 3750 6100 4400
+	6900 1350 9200 1350
+Wire Wire Line
+	9200 1350 9200 2900
+Wire Wire Line
+	9200 2900 8950 2900
+$Comp
+L VMM #PWR034
+U 1 1 5C08852F
+P 9800 2750
+F 0 "#PWR034" H 9800 2600 50  0001 C CNN
+F 1 "VMM" H 9800 2900 50  0000 C CNN
+F 2 "" H 9800 2750 50  0001 C CNN
+F 3 "" H 9800 2750 50  0001 C CNN
+	1    9800 2750
+	1    0    0    -1
+$EndComp
+Wire Wire Line
+	9800 2750 9800 3000
+Wire Wire Line
+	9800 3000 9950 3000
+$Comp
+L Conn_01x02_Female J7
+U 1 1 5C088B80
+P 10700 3950
+F 0 "J7" H 10650 3750 50  0000 C CNN
+F 1 "Conn_01x02_Female" H 10950 4050 50  0000 C CNN
+F 2 "Connectors_Terminal_Blocks:TerminalBlock_bornier-2_P5.08mm" H 10700 3950 50  0001 C CNN
+F 3 "" H 10700 3950 50  0001 C CNN
+	1    10700 3950
+	1    0    0    1
+$EndComp
+$Comp
+L GND #PWR035
+U 1 1 5C089120
+P 10350 4000
+F 0 "#PWR035" H 10350 3750 50  0001 C CNN
+F 1 "GND" H 10350 3850 50  0000 C CNN
+F 2 "" H 10350 4000 50  0001 C CNN
+F 3 "" H 10350 4000 50  0001 C CNN
+	1    10350 4000
+	1    0    0    -1
+$EndComp
+$Comp
+L VDD #PWR036
+U 1 1 5C08917F
+P 10350 3800
+F 0 "#PWR036" H 10350 3650 50  0001 C CNN
+F 1 "VDD" H 10350 3950 50  0000 C CNN
+F 2 "" H 10350 3800 50  0001 C CNN
+F 3 "" H 10350 3800 50  0001 C CNN
+	1    10350 3800
+	1    0    0    -1
+$EndComp
+Wire Wire Line
+	10350 3800 10350 3850
+Wire Wire Line
+	10350 3850 10500 3850
+Wire Wire Line
+	10500 3950 10350 3950
+Wire Wire Line
+	10350 3950 10350 4000
+Wire Wire Line
+	6000 2950 6100 2950
+Wire Wire Line
+	6100 2950 6100 2400
 $EndSCHEMATC
